File: ProjectFiles/KiCad/PulseClockMaster/PulseClockMaster.kicad_sch (KiCad schematic)
At the start: 17 parts, among them Q2 ), Q3 (pin_names, U1 stepdown, U2 ESP01, U3 230to24V, U4 LM358

Commit message: update
Other:
- moved on the sheet: R6
Changed lines of the file:
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@@
 	(wire
 		(pts
-			(xy 201.93 66.04) (xy 205.74 66.04)
+			(xy 203.2 66.04) (xy 205.74 66.04)
 		)
 		(stroke
@@
 	(wire
 		(pts
-			(xy 194.31 66.04) (xy 193.04 66.04)
+			(xy 195.58 66.04) (xy 193.04 66.04)
 		)
 		(stroke
@@
 	(symbol
 		(lib_id "Device:R")
-		(at 198.12 66.04 90)
+		(at 199.39 66.04 90)
 		(unit 1)
 		(exclude_from_sim no)
@@
 		(dnp no)
 		(property "Reference" "R6"
-			(at 197.612 61.976 90)
+			(at 198.882 61.976 90)
 			(effects
 				(font
@@
 		)
 		(property "Value" "220"
-			(at 197.612 63.754 90)
+			(at 198.882 63.754 90)
 			(effects
 				(font
@@
 		)
 		(property "Footprint" "Resistor_SMD:R_0805_2012Metric_Pad1.20x1.40mm_HandSolder"
-			(at 198.12 67.818 90)
+			(at 199.39 67.818 90)
 			(effects
 				(font
@@
 		)
 		(property "Datasheet" "~"
-			(at 198.12 66.04 0)
+			(at 199.39 66.04 0)
 			(effects
 				(font
@@
 		)
 		(property "Description" "Resistor"
-			(at 198.12 66.04 0)
+			(at 199.39 66.04 0)
 			(effects
 				(font
@@
 		)
 		(property "Sim.Device" ""
-			(at 198.12 66.04 90)
-			(effects
-				(font
+			(at 199.39 66.04 90)
+			(effects
+				(font

Commit message: PCB & Javascript updates
Parts:
- J1: value ~ -> 230V AC
- J4: value ~ -> out
- Q2: value ) -> BC817
- Q3: value (pin_names -> BC807
- U2: footprint ownFootprints:ESP01_conn -> ownFootprints:ESP01_conn+outline
Connections:
- net +24V: now also U4.5 (+), U4.6 (-)
Other:
- moved on the sheet: U4B
Changed lines of the file:
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@@
 	)
 	(junction
+		(at 138.43 31.75)
+		(diameter 0)
+		(color 0 0 0 0)
+	)
+	(junction
 		(at 115.57 66.04)
 		(diameter 0)
@@
 	(wire
 		(pts
+			(xy 138.43 29.21) (xy 138.43 31.75)
+		)
+		(stroke
+			(width 0)
+			(type default)
+		)
+	)
+	(wire
+		(pts
 			(xy 140.97 53.34) (xy 143.51 53.34)
 		)
@@
 	(wire
 		(pts
+			(xy 138.43 31.75) (xy 139.7 31.75)
+		)
+		(stroke
+			(width 0)
+			(type default)
+		)
+	)
+	(wire
+		(pts
 			(xy 205.74 68.58) (xy 207.01 68.58)
 		)
@@
 	(wire
 		(pts
+			(xy 138.43 36.83) (xy 139.7 36.83)
+		)
+		(stroke
+			(width 0)
+			(type default)
+		)
+	)
+	(wire
+		(pts
 			(xy 214.63 60.96) (xy 215.9 60.96)
 		)
@@
 	(wire
 		(pts
+			(xy 138.43 36.83) (xy 138.43 31.75)
+		)
+		(stroke
+			(width 0)
+			(type default)
+		)
+	)
+	(wire
+		(pts
 			(xy 149.86 72.39) (xy 139.7 72.39)
 		)
@@
 			)
 		)
-		(property "Value" "~"
+		(property "Value" "230V AC"
 			(at 89.535 64.77 0)
 			(effects
@@
 			)
 		)
-		(property "Value" ")"
+		(property "Value" "BC817"
 			(at 206.502 51.308 0)
 			(effects
@@
 	)
 	(symbol
+		(lib_id "power:+24V")
+		(at 138.43 29.21 0)
+		(unit 1)
+		(exclude_from_sim no)
+		(in_bom yes)
+		(on_board yes)
+		(dnp no)
+		(fields_autoplaced yes)
+		(property "Reference" "#PWR018"
+			(at 138.43 33.02 0)
+			(effects
+				(font
+					(size 1.27 1.27)
+				)
+				(hide yes)
+			)
+		)
+		(property "Value" "+24V"
+			(at 138.43 24.13 0)
+			(effects
+				(font
+					(size 1.27 1.27)
+				)
+			)
+		)
+		(property "Footprint" ""
+			(at 138.43 29.21 0)
+			(effects
+				(font
+					(size 1.27 1.27)
+				)
+				(hide yes)
+			)
+		)
+		(property "Datasheet" ""
+			(at 138.43 29.21 0)
+			(effects
+				(font
+					(size 1.27 1.27)
+				)
+				(hide yes)
+			)
+		)
+		(property "Description" "Power symbol creates a global label with name \"+24V\""
+			(at 138.43 29.21 0)
+			(effects
+				(font
+					(size 1.27 1.27)
+				)
+				(hide yes)
+			)
+		)
+		(pin "1"
+		)
+		(instances
+			(project "PulseClockMaster"
+				(path "/53b661e8-ae03-45d7-aac4-f86aa3eaa041"
+					(reference "#PWR018")
+					(unit 1)
+				)
+			)
+		)
+	)
+	(symbol
 		(lib_id "Own_Library:Mini_AC-DC_230_to_24V_Module_Supply_1")
 		(at 105.41 67.31 0)
@@
 	(symbol
 		(lib_id "Amplifier_Operational:LM358_DFN")
-		(at 257.81 114.3 0)
+		(at 147.32 34.29 0)
 		(unit 2)
 		(exclude_from_sim no)
@@
 		(fields_autoplaced yes)
 		(property "Reference" "U4"
-			(at 257.81 104.14 0)
+			(at 147.32 24.13 0)
 			(effects
 				(font
@@
 		)
 		(property "Value" "LM358"
-			(at 257.81 106.68 0)
+			(at 147.32 26.67 0)
 			(effects
 				(font
@@
 		)
 		(property "Footprint" "Package_SO:SOIC-8_3.9x4.9mm_P1.27mm"
-			(at 257.81 114.3 0)
+			(at 147.32 34.29 0)
 			(effects
 				(font
@@
 		)
 		(property "Datasheet" "www.st.com/resource/en/datasheet/lm358.pdf"
-			(at 257.81 114.3 0)
+			(at 147.32 34.29 0)
 			(effects
 				(font
@@
 		)
 		(property "Description" "Low-Power, Dual Operational Amplifiers, DFN-8"
-			(at 257.81 114.3 0)
+			(at 147.32 34.29 0)
 			(effects
 				(font
@@
 		)
 		(property "Sim.Device" ""
-			(at 257.81 114.3 0)
+			(at 147.32 34.29 0)
 			(effects
 				(font
@@
 		(on_board yes)
 		(dnp no)
-		(fields_autoplaced yes)
 		(property "Reference" "U2"
-			(at 158.115 80.01 0)
+			(at 157.734 67.818 0)
 			(effects
 				(font
@@
 		)
 		(property "Value" "ESP01"
-			(at 158.115 81.28 0)
+			(at 162.052 58.928 0)
 			(effects
 				(font
@@
 			)
 		)
-		(property "Footprint" "ownFootprints:ESP01_conn"
+		(property "Footprint" "ownFootprints:ESP01_conn+outline"
 			(at 157.48 59.69 0)
 			(effects
@@
 			)
 		)
-		(property "Value" "(pin_names"
+		(property "Value" "BC807"
 			(at 206.502 79.756 0)
 			(effects
@@
 			)
 		)
-		(property "Value" "~"
+		(property "Value" "out"
 			(at 224.79 68.5799 0)
 			(effects
