File: ProjectFiles/KiCad/PulseClockMaster/PulseClockMaster.kicad_pcb (KiCad board)
At the start: 2 copper layers, 50 x 43.2 mm, 17 parts, among them Q2 ), Q3 (pin_names, U1 stepdown, U2 ESP01, U3 230to24V, U4 LM358

Commit message: update
Parts:
- moved J4 1.82 mm to (191.0, 42.3)
- moved C2 0.76 mm to (181.9, 43.2)
- moved C1 0.25 mm to (171.2, 43.2)
Routing:
- net +24V: track 48.5 -> 44.9 mm
- net Net-(Q2-E): track 33.7 -> 31.7 mm
- net GND: track 107.7 -> 109.5 mm
- net Net-(J4-Pin_2): track 34.4 -> 33.8 mm
- net Net-(J1-Pin_1): track 12.5 -> 13.1 mm
Other:
- board text added: "22-12-2025"
- board text added: "Master"
- board text added: "PulseClock Master GZ 22-12-2025"

Commit message: readme update
Other:
- board text removed: "22-12-2025"
- board text removed: "Master"
Changed lines of the file:
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@@
 		(at 175.395 86.868 180)
 		(property "Reference" "U2"
-			(at 0 -0.5 180)
+			(at 16.137 13.51 180)
 			(unlocked yes)
 			(layer "F.SilkS")
@@
 		)
 		(property "Value" "ESP01"
-			(at 0 1 180)
+			(at 16.137 15.01 180)
 			(unlocked yes)
 			(layer "F.Fab")
@@
 		(attr through_hole)
 		(fp_text user "${REFERENCE}"
-			(at 0 2.5 180)
+			(at 16.137 16.51 180)
 			(unlocked yes)
 			(layer "F.Fab")
@@
 		(tags "LED")
 		(property "Reference" "D2"
-			(at 1.27 -3.96 90)
+			(at -2.535 1.016 90)
 			(layer "F.SilkS")
 			(effects
@@
 		(at 171.196 55.352)
 		(property "Reference" "U3"
-			(at -23.1 -10.9 0)
+			(at -17.526 -2.774 0)
 			(unlocked yes)
 			(layer "F.SilkS")
@@
 		)
 		(property "Value" "230to24V"
-			(at -23.1 -9.4 0)
+			(at -1.524 -6.838 0)
 			(unlocked yes)
 			(layer "F.Fab")
@@
 		)
 		(fp_text user "Mini AC230 to 25V module"
-			(at 11 -11.5 0)
+			(at -13.462 6.116 0)
 			(unlocked yes)
 			(layer "F.SilkS")
@@
 		)
 		(fp_text user "${REFERENCE}"
-			(at -23.1 -7.9 0)
+			(at -7.366 -6.076 0)
 			(unlocked yes)
 			(layer "F.Fab")
@@
 	)
 	(gr_text "PulseClock\nMaster\nGZ 22-12-2025"
-		(at 249.428 74.676 0)
-		(layer "B.Cu")
-		(effects
-			(font
-				(size 2.5 2.5)
-				(thickness 0.5)
-				(bold yes)
-			)
-			(justify left bottom mirror)
-		)
-	)
-	(gr_text "Master"
-		(at 267.97 50.546 0)
-		(layer "B.Cu")
-		(effects
-			(font
-				(size 2.5 2.5)
-				(thickness 0.5)
-				(bold yes)
-			)
-			(justify left bottom mirror)
-		)
-	)
-	(gr_text "PulseClock\nMaster\nGZ 22-12-2025"
 		(at 175.768 59.69 0)
 		(layer "B.Cu")
@@
 				(bold yes)
 			)
-			(justify left bottom mirror)
-		)
-	)
-	(gr_text "22-12-2025"
-		(at 267.716 57.658 0)
-		(layer "B.Cu")
-		(effects
-			(font
-				(size 2.5 2.5)
-				(thickness 0.5)
-				(bold yes)
-			)

Commit message: issue in PCB
Parts:
- moved U2 32.9 mm to (172.7, 54.1), turned to 0 degrees
- moved R2 2.54 mm to (180.3, 70.9)
- moved R1 1.78 mm to (180.3, 68.6)
Routing:
- net GND: track 109.5 -> 87.5 mm
- net Net-(U2-IO2): track 74.7 -> 61.1 mm
- net +3.3V: track 51.9 -> 45.3 mm
- net Net-(U2-EN): track 8.33 -> 5.52 mm
- net Net-(U2-RST): track 8.16 -> 5.41 mm

Commit message: PCB & Javascript updates
Parts:
- J1: value ~ -> 230V AC
- J4: value ~ -> out
- Q2: value ) -> BC817
- Q3: value (pin_names -> BC807
- U2: footprint ownFootprints:ESP01_conn -> ownFootprints:ESP01_conn+outline
- moved U1 0.29 mm to (178.8, 64.5)
- turned Q2 to 90 degrees
Connections:
- U4 pad 5: unconnected-(U4B-+-Pad5) -> +24V
- U4 pad 6: unconnected-(U4B---Pad6) -> +24V
Routing:
- net Net-(Q2-B): track 20.5 -> 11.3 mm, vias 2 -> 0
- net +24V: track 44.9 -> 38.5 mm
- net Net-(Q2-E): track 31.7 -> 35.6 mm
- net GND: track 87.5 -> 91.1 mm

Commit message: Readme update, small PCB update
Routing:
- net GND: track 91.1 -> 89.7 mm
Changed lines of the file:
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@@
-	)
-	(segment
-		(start 191.008 47.272)
-		(end 191.008 43.6815)
-		(width 0.8)
-		(layer "B.Cu")
-		(net 1)
 	)
 	(segment
@@
 	)
 	(segment
+		(start 191.516 52.816)
+		(end 191.516 55.032)
+		(width 0.8)
+		(layer "B.Cu")
+		(net 1)
+	)
+	(segment
+		(start 183.2 53.852)
+		(end 183.261 53.913)
+		(width 0.5)
+		(layer "B.Cu")
+		(net 1)
+	)
+	(segment
+		(start 187.96 53.356)
+		(end 191.5 53.356)
+		(width 0.5)
+		(layer "B.Cu")
+		(net 1)
+	)
+	(segment
+		(start 192.954 53.594)
+		(end 197.866 53.594)
+		(width 0.8)
+		(layer "B.Cu")
+		(net 1)
+	)
+	(segment
 		(start 199.505 71.259)
 		(end 195.834 74.93)
@@
 	)
 	(segment
-		(start 191.516 52.816)
-		(end 191.516 55.032)
-		(width 0.8)
-		(layer "B.Cu")
-		(net 1)
-	)
-	(segment
-		(start 183.2 53.852)
-		(end 183.261 53.913)
-		(width 0.5)
-		(layer "B.Cu")
-		(net 1)
-	)
-	(segment
-		(start 187.96 53.356)
-		(end 191.5 53.356)
-		(width 0.5)
-		(layer "B.Cu")
-		(net 1)
-	)
-	(segment
 		(start 183.818 53.356)
 		(end 183.261 53.913)
@@
 	)
 	(segment
-		(start 191.516 47.78)
-		(end 191.008 47.272)
-		(width 0.8)
-		(layer "B.Cu")
-		(net 1)
-	)
-	(segment
-		(start 191.036 43.6535)
-		(end 191.036 42.3125)
-		(width 0.8)
-		(layer "B.Cu")
-		(net 1)
-	)
-	(segment
-		(start 192.954 53.594)
-		(end 197.866 53.594)
+		(start 199.505 55.233)
+		(end 199.505 71.259)
 		(width 0.8)
 		(layer "B.Cu")
@@
 	)
 	(segment
-		(start 191.446 55.102)
-		(end 192.954 53.594)
-		(width 0.8)
-		(layer "B.Cu")
-		(net 1)
-	)
-	(segment
 		(start 197.866 53.594)
 		(end 199.505 55.233)
@@
 	)
 	(segment
-		(start 199.505 55.233)
-		(end 199.505 71.259)
+		(start 191.008 43.6815)
+		(end 191.036 43.6535)
 		(width 0.8)
 		(layer "B.Cu")
@@
 		(end 195.715 75.184)
 		(width 0.8)
-		(layer "B.Cu")
-		(net 1)
-	)
-	(segment
-		(start 191.516 51.437)
-		(end 191.516 52.816)
-		(width 0.5)
 		(layer "B.Cu")
 		(net 1)
@@
 	)
 	(segment
+		(start 191.446 55.102)
+		(end 192.954 53.594)
+		(width 0.8)
+		(layer "B.Cu")
+		(net 1)
+	)
+	(segment
+		(start 191.516 52.816)
+		(end 191.008 52.308)
+		(width 0.8)
+		(layer "B.Cu")
+		(net 1)
+	)
+	(segment
 		(start 179.205 75.692)
 		(end 179.713 75.184)
@@
 	)
 	(segment
+		(start 191.008 52.308)
+		(end 191.008 43.6815)
+		(width 0.8)
+		(layer "B.Cu")
+		(net 1)
+	)
+	(segment
 		(start 191.5 53.356)
 		(end 191.516 53.34)
@@
 	)
 	(segment
-		(start 191.516 52.816)
-		(end 191.516 47.78)
-		(width 0.8)
-		(layer "B.Cu")
-		(net 1)
-	)
-	(segment
 		(start 172.72 74.422)
 		(end 173.99 75.692)
@@
 	)
 	(segment
-		(start 191.008 43.6815)
-		(end 191.036 43.6535)
+		(start 191.036 43.6535)
+		(end 191.036 42.3125)
 		(width 0.8)
 		(layer "B.Cu")
@@
 	)
 	(segment
+		(start 198.501 70.485)
+		(end 196.596 72.39)
+		(width 0.5)
+		(layer "B.Cu")
+		(net 11)
+	)
+	(segment
 		(start 192.9765 57.404)
 		(end 195.1355 57.404)
@@
 	)
 	(segment
+		(start 196.596 72.39)
+		(end 178.562 72.39)
+		(width 0.5)
+		(layer "B.Cu")
+		(net 11)
+	)
+	(segment
+		(start 198.501 60.579)
+		(end 198.501 70.485)
+		(width 0.5)
+		(layer "B.Cu")
+		(net 11)
+	)
+	(segment
 		(start 185.547 55.626)
 		(end 186.817 54.356)
-		(width 0.5)
-		(layer "B.Cu")
-		(net 11)
-	)
-	(segment
-		(start 198.321819 60.399819)
-		(end 198.321819 70.664181)
-		(width 0.5)
-		(layer "B.Cu")
-		(net 11)
-	)
-	(segment
-		(start 173.933 73.095)
-		(end 172.72 71.882)
 		(width 0.5)
 		(layer "B.Cu")
@@
 	(segment
 		(start 195.326 57.404)
-		(end 198.321819 60.399819)
+		(end 198.501 60.579)
 		(width 0.5)
 		(layer "B.Cu")
@@
 	)
 	(segment
-		(start 196.596 72.39)
-		(end 178.562 72.39)
+		(start 178.562 72.39)
+		(end 177.857 73.095)
 		(width 0.5)
 		(layer "B.Cu")
@@
 	)
 	(segment
+		(start 177.857 73.095)
+		(end 173.933 73.095)
+		(width 0.5)
+		(layer "B.Cu")
+		(net 11)
+	)
+	(segment
 		(start 182.118 55.626)
 		(end 185.547 55.626)
@@
 	)
 	(segment
-		(start 198.321819 70.664181)
-		(end 196.596 72.39)
-		(width 0.5)
-		(layer "B.Cu")
-		(net 11)
-	)
-	(segment
-		(start 178.562 72.39)
-		(end 177.857 73.095)
-		(width 0.5)
-		(layer "B.Cu")
-		(net 11)
-	)
-	(segment
-		(start 195.326 57.404)
-		(end 195.072 57.404)
+		(start 173.933 73.095)
+		(end 172.72 71.882)
 		(width 0.5)
 		(layer "B.Cu")
@@
 	)
 	(segment
-		(start 177.857 73.095)
-		(end 173.933 73.095)
-		(width 0.5)
-		(layer "B.Cu")
-		(net 11)
-	)
-	(segment
 		(start 189.23 54.356)
 		(end 189.806079 54.932079)
@@
 		(width 0.5)
 		(layer "B.Cu")
+		(net 11)
+	)
+	(segment
+		(start 195.072 57.404)
+		(end 195.326 57.404)
+		(width 0.5)
+		(layer "B.Cu")

Commit message: some cleanup
Parts:
- moved J1 1.05 mm to (157.3, 41.4)
- moved J4 1.05 mm to (191.3, 41.3)
Routing:
- net Net-(J1-Pin_2): track 20.1 -> 21.2 mm
- net Net-(J1-Pin_1): track 13.1 -> 14.1 mm
- net GND: track 89.7 -> 90.7 mm
Changed lines of the file:
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@@
 	(footprint "TerminalBlock:TerminalBlock_MaiXu_MX126-5.0-02P_1x02_P5.00mm"
 		(layer "F.Cu")
-		(at 157.306 42.418)
+		(at 157.306 41.3695)
 		(descr "terminal block MaiXu MX126-5.0-02P, 2 pins, pitch 5mm, size 10.5x7.8mm, drill diameter 1.3mm, pad diameter 2.8mm, https://www.lcsc.com/datasheet/lcsc_datasheet_2309150913_MAX-MX126-5-0-03P-GN01-Cu-S-A_C5188435.pdf, script-generated using https://gitlab.com/kicad/libraries/kicad-footprint-generator/-/tree/master/scripts/TerminalBlock_MaiXu")
 		(tags "THT terminal block MaiXu MX126-5.0-02P pitch 5mm size 10.5x7.8mm drill 1.3mm pad 2.8mm")
@@
 	(footprint "TerminalBlock_4Ucon:TerminalBlock_4Ucon_1x02_P3.50mm_Horizontal"
 		(layer "F.Cu")
-		(at 191.036 42.3125)
+		(at 191.29 41.2965)
 		(descr "Terminal Block 4Ucon ItemNo. 19963, 2 pins, pitch 3.5mm, size 7.7x7mm, drill diameter 1.2mm, pad diameter 2.4mm, http://www.4uconnector.com/online/object/4udrawing/19963.pdf, script-generated using https://gitlab.com/kicad/libraries/kicad-footprint-generator/-/tree/master/scripts/TerminalBlock_4Ucon")
 		(tags "THT Terminal Block 4Ucon ItemNo. 19963 pitch 3.5mm size 7.7x7mm drill 1.2mm pad 2.4mm")
@@
 		(tags "CP Radial series Radial pin pitch 3.80mm diameter 8mm height 14mm Electrolytic Capacitor")
 		(property "Reference" "C1"
-			(at 1.9 -5.25 90)
+			(at 2.9485 -5.25 90)
 			(layer "F.SilkS")
 			(effects
@@
 		(tags "resistor handsolder")
 		(property "Reference" "R1"
-			(at 0 1.65 0)
+			(at -2.667 -0.254 0)
 			(layer "B.SilkS")
 			(effects
@@
 		)
 		(fp_text user "${REFERENCE}"
-			(at 0 0 0)
+			(at -2.413 0 0)
 			(layer "B.Fab")
 			(effects
@@
 		(tags "SOT TO_SOT_SMD")
 		(property "Reference" "Q2"
-			(at 0 2.4 90)
+			(at -3.3805 -2.347 90)
 			(layer "B.SilkS")
 			(effects
@@
 		(tags "resistor handsolder")
 		(property "Reference" "R2"
-			(at 0 1.65 0)
+			(at -2.794 0.254 0)
 			(layer "B.SilkS")
 			(effects
@@
 		)
 		(fp_text user "${REFERENCE}"
-			(at 0 0 0)
+			(at -2.413 0 0)
 			(layer "B.Fab")
 			(effects
@@
 		)
 		(property "Value" "BC807"
-			(at 0 -2.4 90)
+			(at -0.508 2.982 90)
 			(layer "B.Fab")
 			(effects
@@
 	)
 	(segment
-		(start 191.516 55.032)
-		(end 191.446 55.102)
-		(width 0.8)
-		(layer "B.Cu")
-		(net 1)
-	)
-	(segment
 		(start 185.801 49.022)
 		(end 187.071 49.022)
@@
 	)
 	(segment
-		(start 191.516 52.816)
-		(end 191.516 55.032)
-		(width 0.8)
-		(layer "B.Cu")
-		(net 1)
-	)
-	(segment
 		(start 183.2 53.852)
 		(end 183.261 53.913)
@@
 	)
 	(segment
+		(start 191.446 55.102)
+		(end 191.516 55.032)
+		(width 0.8)
+		(layer "B.Cu")
+		(net 1)
+	)
+	(segment
+		(start 191.262 52.562)
+		(end 191.262 51.292)
+		(width 0.8)
+		(layer "B.Cu")
+		(net 1)
+	)
+	(segment
 		(start 183.818 53.356)
 		(end 183.261 53.913)
@@
 	)
 	(segment
+		(start 191.516 52.816)
+		(end 191.262 52.562)
+		(width 0.8)
+		(layer "B.Cu")
+		(net 1)
+	)
+	(segment
 		(start 199.505 55.233)
 		(end 199.505 71.259)
@@
 	)
 	(segment
-		(start 191.008 43.6815)
-		(end 191.036 43.6535)
+		(start 191.262 42.6655)
+		(end 191.29 42.6375)
 		(width 0.8)
 		(layer "B.Cu")
@@
 	)
 	(segment
-		(start 191.008 43.561)
-		(end 191.008 41.275)
+		(start 191.262 42.545)
+		(end 191.262 40.259)
 		(width 2.8)
 		(layer "B.Cu")
@@
 	)
 	(segment
-		(start 191.446 55.102)
-		(end 192.954 53.594)
+		(start 191.516 55.032)
+		(end 191.516 52.816)
 		(width 0.8)
 		(layer "B.Cu")
@@
 	)
 	(segment
-		(start 191.516 52.816)
-		(end 191.008 52.308)
+		(start 191.446 55.102)
+		(end 192.954 53.594)
 		(width 0.8)
 		(layer "B.Cu")
@@
 	)
 	(segment
-		(start 191.008 52.308)
-		(end 191.008 43.6815)
+		(start 191.262 51.292)
+		(end 191.262 42.6655)
 		(width 0.8)
 		(layer "B.Cu")
@@
 	)
 	(segment
-		(start 191.036 43.6535)
-		(end 191.036 42.3125)
+		(start 191.29 42.6375)
+		(end 191.29 41.2965)
 		(width 0.8)
 		(layer "B.Cu")
@@
 	)
 	(segment
-		(start 157.226 43.434)
-		(end 157.226 41.148)
+		(start 157.226 42.3855)
+		(end 157.226 40.0995)
 		(width 2.8)
 		(layer "B.Cu")
@@
 	)
 	(segment
-		(start 157.306 42.418)
+		(start 157.306 41.3695)
 		(end 157.306 48.18)
 		(width 0.8)
@@
 	)
 	(segment
-		(start 198.501 70.485)
-		(end 196.596 72.39)
-		(width 0.5)
-		(layer "B.Cu")
-		(net 11)
-	)
-	(segment
 		(start 192.9765 57.404)
 		(end 195.1355 57.404)
@@
 	)
 	(segment
-		(start 196.596 72.39)
-		(end 178.562 72.39)
+		(start 190.5 57.404)
+		(end 193.04 57.404)
 		(width 0.5)
 		(layer "B.Cu")
@@
 	)
 	(segment
-		(start 198.501 60.579)
-		(end 198.501 70.485)
+		(start 195.072 57.404)
+		(end 195.58 57.404)
 		(width 0.5)
 		(layer "B.Cu")
@@
 	)
 	(segment
-		(start 181.991 55.499)
-		(end 182.118 55.626)
+		(start 198.501 70.485)
+		(end 196.596 72.39)
 		(width 0.5)
 		(layer "B.Cu")
@@
 	)
 	(segment
-		(start 172.72 71.882)
-		(end 171.704 71.882)
-		(width 1.5)
+		(start 198.501 60.325)
+		(end 198.501 70.485)
+		(width 0.5)
 		(layer "B.Cu")
 		(net 11)
 	)
 	(segment
-		(start 195.326 57.404)
-		(end 198.501 60.579)
+		(start 195.58 57.404)
+		(end 198.501 60.325)
 		(width 0.5)
 		(layer "B.Cu")
@@
 	)
 	(segment
-		(start 187.071 54.356)
-		(end 189.23 54.356)
-		(width 0.4)
+		(start 181.991 55.499)
+		(end 182.118 55.626)
+		(width 0.5)
 		(layer "B.Cu")
 		(net 11)
 	)
 	(segment
-		(start 178.562 72.39)
-		(end 177.857 73.095)
-		(width 0.5)
+		(start 172.72 71.882)
+		(end 171.704 71.882)
+		(width 1.5)
 		(layer "B.Cu")
 		(net 11)
 	)
 	(segment
-		(start 190.246 57.404)
-		(end 193.04 57.404)
+		(start 178.562 72.39)
+		(end 177.857 73.095)
 		(width 0.5)
 		(layer "B.Cu")
@@
 	)
 	(segment
-		(start 177.857 73.095)
-		(end 173.933 73.095)
-		(width 0.5)
+		(start 187.071 54.356)
+		(end 189.23 54.356)
+		(width 0.4)
 		(layer "B.Cu")
 		(net 11)
@@
 	)
 	(segment
-		(start 173.933 73.095)
-		(end 172.72 71.882)
+		(start 177.857 73.095)
+		(end 173.933 73.095)
 		(width 0.5)
 		(layer "B.Cu")
@@
 	)
 	(segment
-		(start 189.806079 56.964079)
-		(end 190.246 57.404)
+		(start 189.23 54.356)
+		(end 189.806079 54.932079)
 		(width 0.5)
 		(layer "B.Cu")
@@
 	)
 	(segment
-		(start 189.23 54.356)
-		(end 189.806079 54.932079)
+		(start 189.806079 54.932079)
+		(end 189.806079 56.710079)
 		(width 0.5)
 		(layer "B.Cu")
@@
 	)
 	(segment
-		(start 189.806079 54.932079)
-		(end 189.806079 56.964079)
+		(start 173.933 73.095)
+		(end 172.72 71.882)
 		(width 0.5)
 		(layer "B.Cu")
@@
 	)
 	(segment
-		(start 195.072 57.404)
-		(end 195.326 57.404)
+		(start 196.596 72.39)
+		(end 178.562 72.39)
+		(width 0.5)
+		(layer "B.Cu")
+		(net 11)
+	)
+	(segment
+		(start 189.806079 56.710079)
+		(end 190.5 57.404)
 		(width 0.5)
 		(layer "B.Cu")
@@
 	)
 	(segment
-		(start 194.564 39.878)
-		(end 194.564 40.1255)
+		(start 194.818 39.1095)
+		(end 194.79 39.1375)
 		(width 0.8)
 		(layer "B.Cu")
@@
 	)
 	(segment
-		(start 194.536 40.1535)
-		(end 194.536 42.3125)
+		(start 170.942 39.38)
+		(end 182.626 39.38)
 		(width 0.8)
 		(layer "B.Cu")
@@
 	)
 	(segment
-		(start 192.024 37.338)
-		(end 194.564 39.878)
-		(width 0.8)
+		(start 170.18 39.37)
+		(end 171.958 39.37)
+		(width 1.5)
 		(layer "B.Cu")
 		(net 16)
@@
 	(segment
 		(start 182.626 39.38)
-		(end 184.668 37.338)
+		(end 185.176 36.83)
 		(width 0.8)
 		(layer "B.Cu")
@@
 	)
 	(segment
-		(start 170.18 39.37)
-		(end 171.958 39.37)
-		(width 1.5)
+		(start 194.818 42.545)
+		(end 194.818 40.259)
+		(width 2.8)
 		(layer "B.Cu")
 		(net 16)
 	)
 	(segment
-		(start 194.564 40.1255)
-		(end 194.536 40.1535)
+		(start 192.786 36.83)
+		(end 194.818 38.862)
 		(width 0.8)
 		(layer "B.Cu")
@@
 	)
 	(segment
-		(start 194.564 43.561)
-		(end 194.564 41.275)
-		(width 2.8)
+		(start 194.79 39.1375)
+		(end 194.79 41.2965)
+		(width 0.8)
 		(layer "B.Cu")
 		(net 16)
 	)
 	(segment
-		(start 170.942 39.38)
-		(end 182.626 39.38)
+		(start 185.176 36.83)
+		(end 192.786 36.83)
 		(width 0.8)
 		(layer "B.Cu")
@@
 	)
 	(segment
-		(start 184.668 37.338)
-		(end 192.024 37.338)
+		(start 194.818 38.862)
+		(end 194.818 39.1095)
 		(width 0.8)
 		(layer "B.Cu")
@@
 	)
 	(segment
-		(start 162.306 43.434)
-		(end 162.306 41.148)
+		(start 162.306 42.3855)
+		(end 162.306 40.0995)
 		(width 2.8)
 		(layer "B.Cu")
@@
 	(segment
 		(start 162.306 47.752)
-		(end 162.306 42.418)
+		(end 162.306 41.3695)
 		(width 0.8)
 		(layer "B.Cu")
